File: Hardware/proyecto de paneles solares/proyecto de paneles solares.kicad_pcb (KiCad board)
At the start: 2 copper layers, 14 parts, among them J1 Conn_01x04, J2 Conn_01x02, J4 Screw_Terminal_01x02, U1 ESP32-DEVKIT-V1, U2 TP4056_MICRO-USB_CHARGER_-_1A, U3 AMS1117-3.3

Commit message: Add files via upload
Parts:
- removed J2: Conn_01x02, Connector_PinHeader_2.54mm:PinHeader_1x02_P2.54mm_Vertical
- added J3: Screw_Terminal_01x02, TerminalBlock:TerminalBlock_MaiXu_MX126-5.0-02P_1x02_P5.00mm, F.Cu at (104.2, 112.0)
Connections:
- C2 pad 1: GND -> Net-(U1-3V3)
- C2 pad 2: Net-(U1-3V3) -> GND
