File: Hardware/proyecto de paneles solares/proyecto de paneles solares.kicad_sch (KiCad schematic)
At the start: 14 parts, among them J1 Conn_01x04, J2 Conn_01x02, J4 Screw_Terminal_01x02, U1 ESP32-DEVKIT-V1, U2 TP4056_MICRO-USB_CHARGER_-_1A, U3 AMS1117-3.3

Commit message: Add files via upload
Parts:
- removed J2: Conn_01x02, Connector_PinHeader_2.54mm:PinHeader_1x02_P2.54mm_Vertical, symbol Connector_Generic:Conn_01x02
- added J3: Screw_Terminal_01x02, TerminalBlock:TerminalBlock_MaiXu_MX126-5.0-02P_1x02_P5.00mm, symbol Connector:Screw_Terminal_01x02
Connections:
- net GND: now also J3.1 (Pin_1)
- net at Diodo_1N5819.2 (A): now also J3.2 (Pin_2)
Changed lines of the file:
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@@
 	)
 	(symbol
-		(lib_id "Connector_Generic:Conn_01x02")
-		(at 92.71 44.45 0)
-		(mirror y)
+		(lib_id "Connector:Screw_Terminal_01x02")
+		(at 92.71 46.99 180)
 		(unit 1)
 		(exclude_from_sim no)
@@
 		(on_board yes)
 		(dnp no)
-		(property "Reference" "J2"
-			(at 92.71 53.34 0)
+		(fields_autoplaced yes)
+		(property "Reference" "J3"
+			(at 92.71 38.1 0)
 			(effects
 				(font
@@
 			)
 		)
-		(property "Value" "Conn_01x02"
-			(at 92.71 50.8 0)
+		(property "Value" "Screw_Terminal_01x02"
+			(at 92.71 40.64 0)
 			(effects
 				(font
@@
 			)
 		)
-		(property "Footprint" "Connector_PinHeader_2.54mm:PinHeader_1x02_P2.54mm_Vertical"
-			(at 92.71 44.45 0)
+		(property "Footprint" "TerminalBlock:TerminalBlock_MaiXu_MX126-5.0-02P_1x02_P5.00mm"
+			(at 92.71 46.99 0)
 			(effects
 				(font
@@
 		)
 		(property "Datasheet" "~"
-			(at 92.71 44.45 0)
+			(at 92.71 46.99 0)
 			(effects
 				(font
@@
 			)
 		)
-		(property "Description" "Generic connector, single row, 01x02, script generated (kicad-library-utils/schlib/autogen/connector/)"
-			(at 92.71 44.45 0)
+		(property "Description" "Generic screw terminal, single row, 01x02, script generated (kicad-library-utils/schlib/autogen/connector/)"
+			(at 92.71 46.99 0)
 			(effects
 				(font
@@
 			)
 		)
+		(pin "1"
+		)
 		(pin "2"
-		)
-		(pin "1"
 		)
 		(instances
 			(project ""
 				(path "/1cbbe343-2e72-4edf-9641-106025a9c0b7"
-					(reference "J2")
+					(reference "J3")
 					(unit 1)
 				)
